File: SolarSense_v1.kicad_sch (KiCad schematic)
At the start: 40 parts, among them IC1 HT7833, J1 Conn_01x04_Pin, J2 Conn_01x04_Pin, J3 KF141R-2.54-2P, J4 BWSMA-KE-P001, J6 U.FL-R-SMT_01_, J7 KF141R-2.54-2P, U1 MCP1640T-I_CHY, U3 TP4056, U4 LoRa-E5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

Commit message: First routing
Connections:
- net CURRENT_SENSOR: now also U4.27 (PA10); no longer U4.7 (PB4)
- net LED: now also U4.20 (PB10); no longer U4.21 (PA9)
- net RX: now also J1.3 (Pin_3); no longer J1.2 (Pin_2)
- net STEP-UP-EN: now also U4.21 (PA9); no longer U4.20 (PB10)
- net TX: now also J1.2 (Pin_2); no longer J1.3 (Pin_3)
- net BAT_VOLTAGE: no longer names the net of U4.8 (PB3)
- no-connect marks 19 -> 20
Changed lines of the file:
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@@
   (no_connect (at 120.65 60.96))
   (no_connect (at 93.98 189.23))
+  (no_connect (at 95.25 78.74))
   (no_connect (at 105.41 78.74))
   (no_connect (at 107.95 78.74))
   (no_connect (at 102.87 43.18))
-  (no_connect (at 97.79 43.18))
   (no_connect (at 243.84 148.59))
   (no_connect (at 120.65 63.5))
@@
   (no_connect (at 107.95 43.18))
   (no_connect (at 120.65 58.42))
+  (no_connect (at 85.09 68.58))
   (wire (pts (xy 29.21 181.61) (xy 38.1 181.61))
     (stroke (width 0) (type default))
@@
     (stroke (width 0) (type default))
   )
-  (wire (pts (xy 76.2 68.58) (xy 85.09 68.58))
-    (stroke (width 0) (type default))
-  )
   (wire (pts (xy 50.8 63.5) (xy 54.61 63.5))
     (stroke (width 0) (type default))
@@
     (stroke (width 0) (type default))
   )
+  (wire (pts (xy 97.79 36.83) (xy 97.79 43.18))
+    (stroke (width 0) (type default))
+  )
   (wire (pts (xy 48.26 181.61) (xy 55.88 181.61))
     (stroke (width 0) (type default))
@@
   )
   (wire (pts (xy 93.98 201.93) (xy 91.44 201.93))
-    (stroke (width 0) (type default))
-  )
-  (wire (pts (xy 95.25 83.82) (xy 95.25 78.74))
     (stroke (width 0) (type default))
   )
@@
     (effects (font (size 2 2) (thickness 0.254) bold) (justify left bottom))
   )
-  (text "add = 0b1001000" (at 256.54 82.55 0)
+  (text "add = 0b1001000" (at 260.35 59.69 0)
     (effects (font (size 1.27 1.27)) (justify left bottom))
   )
@@
     )
   )
-  (global_label "STEP-UP-EN" (shape input) (at 128.27 55.88 0) (fields_autoplaced)
-    (effects (font (size 1.27 1.27)) (justify left))
-    (property "Intersheetrefs" "${INTERSHEET_REFS}" (at 144.0761 55.88 0)
+  (global_label "STEP-UP-EN" (shape input) (at 128.27 53.34 0) (fields_autoplaced)
+    (effects (font (size 1.27 1.27)) (justify left))
+    (property "Intersheetrefs" "${INTERSHEET_REFS}" (at 144.0761 53.34 0)
       (effects (font (size 1.27 1.27)) (justify left) hide)
     )
@@
     )
   )
-  (global_label "RX" (shape input) (at 153.67 196.85 0) (fields_autoplaced)
-    (effects (font (size 1.27 1.27)) (justify left))
-    (property "Intersheetrefs" "${INTERSHEET_REFS}" (at 159.1347 196.85 0)
-      (effects (font (size 1.27 1.27)) (justify left) hide)
-    )
-  )
-  (global_label "TX" (shape input) (at 153.67 199.39 0) (fields_autoplaced)
-    (effects (font (size 1.27 1.27)) (justify left))
-    (property "Intersheetrefs" "${INTERSHEET_REFS}" (at 158.8323 199.39 0)
+  (global_label "RX" (shape input) (at 153.67 199.39 0) (fields_autoplaced)
+    (effects (font (size 1.27 1.27)) (justify left))
+    (property "Intersheetrefs" "${INTERSHEET_REFS}" (at 159.1347 199.39 0)
+      (effects (font (size 1.27 1.27)) (justify left) hide)
+    )
+  )
+  (global_label "TX" (shape input) (at 153.67 196.85 0) (fields_autoplaced)
+    (effects (font (size 1.27 1.27)) (justify left))
+    (property "Intersheetrefs" "${INTERSHEET_REFS}" (at 158.8323 196.85 0)
       (effects (font (size 1.27 1.27)) (justify left) hide)
     )
@@
     )
   )
-  (global_label "CURRENT_SENSOR" (shape input) (at 76.2 68.58 180) (fields_autoplaced)
-    (effects (font (size 1.27 1.27)) (justify right))
-    (property "Intersheetrefs" "${INTERSHEET_REFS}" (at 56.1606 68.58 0)
-      (effects (font (size 1.27 1.27)) (justify right) hide)
-    )
-  )
-  (global_label "BAT_VOLTAGE" (shape input) (at 95.25 83.82 270) (fields_autoplaced)
-    (effects (font (size 1.27 1.27)) (justify right))
-    (property "Intersheetrefs" "${INTERSHEET_REFS}" (at 95.25 99.0214 90)
-      (effects (font (size 1.27 1.27)) (justify right) hide)
+  (global_label "CURRENT_SENSOR" (shape input) (at 97.79 36.83 90) (fields_autoplaced)
+    (effects (font (size 1.27 1.27)) (justify left))
+    (property "Intersheetrefs" "${INTERSHEET_REFS}" (at 97.79 16.7906 90)
+      (effects (font (size 1.27 1.27)) (justify left) hide)
     )
   )
@@
     )
   )
-  (global_label "LED" (shape input) (at 128.27 53.34 0) (fields_autoplaced)
-    (effects (font (size 1.27 1.27)) (justify left))
-    (property "Intersheetrefs" "${INTERSHEET_REFS}" (at 134.7023 53.34 0)
-      (effects (font (size 1.27 1.27)) (justify left) hide)
-    )
+  (global_label "LED" (shape input) (at 128.27 55.88 0) (fields_autoplaced)
+    (effects (font (size 1.27 1.27)) (justify left))
+    (property "Intersheetrefs" "${INTERSHEET_REFS}" (at 134.7023 55.88 0)
+      (effects (font (size 1.27 1.27)) (justify left) hide)
+    )
